File: Micromouse/Micromouse.sch (KiCad schematic (older format))
At the start: 11 parts

Commit message: finished schamtic
Parts:
- added R1, R2, R3, R4, R5, R6: R, symbol Device:R
- added SW1, SW2: Encoder, symbol motor_encoder:Encoder
- IC1: renamed from IC?; symbol SN754410:SN754410 -> Micromouse-rescue:SN754410-SN754410
- U1: renamed from U?; symbol Teensy:Teensy3.2 -> Micromouse-rescue:Teensy3.2-Teensy
- gave numbers to parts that had none: 6
Connections:
- net labels added: 1.8K, 5V, D0, D1, D17, D18, D2
- wire segments 29 -> 52
Other:
- moved on the sheet: D1, D2, D3, IC1, M1, M2, Q?

Commit message: finished schematic
Connections:
- net labels added: 120
Changed lines of the file:
@@
 Wire Wire Line
 	6350 2550 6850 2550
+Text Label 1100 1450 0    50   ~ 0
+120
 $EndSCHEMATC

Commit message: labels to resistors
Connections:
- net labels removed: 1.8K, 120
Other:
- note added: "R1-3 = 1.8kΩ\n"
- note added: "R4-6 = 120Ω\n"
Changed lines of the file:
@@
 Wire Wire Line
 	3150 1800 3850 1800
-Text Label 1250 2050 2    50   ~ 0
-1.8K
 $Comp
 L Device:R R4
@@
 Wire Wire Line
 	6350 2550 6850 2550
-Text Label 1100 1450 0    50   ~ 0
-120
+Text Notes 650  2100 0    50   ~ 0
+R1-3 = 1.8kΩ\n
+Text Notes 700  1400 0    50   ~ 0
+R4-6 = 120Ω\n
 $EndSCHEMATC
